File: hw4/PIC_PCB/PIC_PCB.kicad_pcb (KiCad board)
At the start: 2 copper layers, 60 x 60 mm, 23 parts, among them J1 Battery, J2 Conn_01x06_Male, J3 Left, J4 Right, SW1 SW_Slide, SW2 RESET, SW3 USER, U1 AP7381-33V, U2 PIC32MX170F256B

Commit message: Finished PCB
Routing:
- net +3V3: track 96.8 -> 163.4 mm
- net /RESET: track 0.00 -> 66.2 mm
- net /USER: track 0.00 -> 65.5 mm, vias 0 -> 1
- net /YELLOW: track 0.00 -> 57.0 mm, vias 0 -> 1
- net /GREEN: track 0.00 -> 54.1 mm, vias 0 -> 1
- net /B13: track 0.00 -> 39.1 mm
- net /U1TX: track 0.00 -> 34.0 mm
- net /B7: track 0.00 -> 31.3 mm, vias 0 -> 2
- net /B9: track 0.00 -> 31.3 mm
- net /B8: track 0.00 -> 31.3 mm
- net /U1RX: track 0.00 -> 31.1 mm
- net /B15: track 0.00 -> 29.2 mm
- net /B14: track 0.00 -> 29.2 mm
- net /B12: track 0.00 -> 29.2 mm
- net /B11: track 0.00 -> 29.2 mm
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